File: kiCadFiles/Calibration-PCB-1.kicad_pcb (KiCad board)
At the start: 2 copper layers, 78.7 x 88.9 mm, 25 parts, among them J1 Raspberry_Pi_2_3, J2 Screw_Terminal_01x02, U1 OPA552P, U2 OPA552P, U3 OPA552P, U4 OPA552P, U5 OPA552P, U6 OPA552P, U7 RJHSE538103

Commit message: Add files via upload
Parts:
- removed the REF** at (160.0, 86.4)
- moved REF** 1.27 mm to (160.0, 146.1)
Other:
- board size 78.7 x 88.9 mm -> 78.8 x 88.9 mm
Changed lines of the file:
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@@
   )
   (footprint "MountingHole:MountingHole_2.7mm_Pad" (layer "F.Cu")
-    (at 160.02 147.32)
+    (at 160.02 146.05)
     (descr "Mounting Hole 2.7mm")
     (tags "mounting hole 2.7mm")
@@
     )
   )
-  (footprint "MountingHole:MountingHole_2.7mm_Pad" (layer "F.Cu")
-    (at 160.02 86.36)
-    (descr "Mounting Hole 2.7mm")
-    (tags "mounting hole 2.7mm")
-    (attr exclude_from_pos_files exclude_from_bom)
-    (fp_text reference "REF**" (at 0 -3.7) (layer "F.SilkS") hide
-        (effects (font (size 1 1) (thickness 0.15)))
-    )
-    (fp_text value "MountingHole_2.7mm_Pad" (at 0 3.7) (layer "F.Fab")
-        (effects (font (size 1 1) (thickness 0.15)))
-    )
-    (fp_text user "${REFERENCE}" (at 0 0) (layer "F.Fab")
-        (effects (font (size 1 1) (thickness 0.15)))
-    )
-    (fp_circle (center 0 0) (end 2.7 0)
-      (stroke (width 0.15) (type solid)) (fill none) (layer "Cmts.User"))
-    (fp_circle (center 0 0) (end 2.95 0)
-      (stroke (width 0.05) (type solid)) (fill none) (layer "F.CrtYd"))
-    (pad "1" thru_hole circle (at 0 0) (size 5.4 5.4) (drill 2.7) (layers *.Cu *.Mask))
-  )
-  (gr_arc (start 162.56 81.28) (mid 164.356051 82.023949) (end 165.1 83.82)
+  (gr_arc (start 162.56 86.36) (mid 164.453607 87.006393) (end 165.1 88.9)
     (stroke (width 0.05) (type default)) (layer "Edge.Cuts"))
   (gr_line (start 86.36 139.7) (end 86.36 76.2)
     (stroke (width 0.05) (type default)) (layer "Edge.Cuts"))
-  (gr_line (start 165.1 83.82) (end 165.1 86.36)
+  (gr_line (start 154.94 83.82) (end 154.94 86.36)
     (stroke (width 0.05) (type default)) (layer "Edge.Cuts"))
   (gr_arc (start 86.36 66.04) (mid 87.103949 64.243949) (end 88.9 63.5)
@@
   (gr_line (start 104.14 63.5) (end 93.98 63.5)
     (stroke (width 0.05) (type default)) (layer "Edge.Cuts"))
-  (gr_line (start 154.94 81.28) (end 162.56 81.28)
+  (gr_line (start 154.94 86.36) (end 162.56 86.36)
     (stroke (width 0.05) (type default)) (layer "Edge.Cuts"))
   (gr_line (start 93.98 63.5) (end 91.44 63.5)
@@
   (gr_arc (start 152.4 63.5) (mid 154.196051 64.243949) (end 154.94 66.04)
     (stroke (width 0.05) (type default)) (layer "Edge.Cuts"))
-  (gr_line (start 165.1 88.9) (end 165.1 86.36)
+  (gr_line (start 154.94 83.82) (end 154.94 81.28)
     (stroke (width 0.05) (type default)) (layer "Edge.Cuts"))
   (gr_line (start 165.1 88.9) (end 165.1 142.24)
@@
   )
   (target plus (at 91.44 147.32) (size 5) (width 0.05) (layer "Edge.Cuts"))
-  (target plus (at 160.02 86.36) (size 5) (width 0.05) (layer "Edge.Cuts"))
-  (target plus (at 160.02 147.32) (size 5) (width 0.05) (layer "Edge.Cuts"))
+  (target plus (at 160.02 146.05) (size 5) (width 0.05) (layer "Edge.Cuts"))
   (target plus (at 91.44 68.58) (size 5) (width 0.05) (layer "Edge.Cuts"))
   (segment (start 97.8 118.1) (end 99.08 119.38) (width 0.25) (layer "F.Cu") (net 1))
